File: KiCAD/JU-TE-6K-Video-HW-Patch.kicad_sch (KiCad schematic)
At the start: 3 parts, among them U1 DL030D, U2 DL004D, U3 DL000D

Commit message: Update
Parts:
- added unit 6 of U2
- added unit 5 of U2
Connections:
- net CPU_WAIT: now also U2.12 (Y6); no longer U3.2 (B1), U3.6 (Y2)
- net D14-Y2 (DL295) : now also U2.3 (A2); no longer U2.5 (A3)
- net STOP_CPU_WAIT: now also U2.4 (Y2); no longer U2.6 (Y3)
- new net: U2.11 (A5), U3.2 (B1), U3.6 (Y2)
- new net: U2.10 (Y5), U2.13 (A6)
Other:
- note added: "Erkennung T1-State der Host-CPU bei Zugriff auf den BWS (4000H-5FFFH)"
- note added: "Verzögerung"
- note removed: "Erkennung T1-State der Host-CPU bei Zugriff auf IRM (4000H-5FFFH)"
- title: Ju-TeC 6K Video-Entstörung -> JU-TE 6K Video-Entstörung
- moved on the sheet: U3A, U3B, U3C

Commit message: Booster Switch update
Parts:
- added R102: 10K, symbol Device:R
- added SW1: ~, symbol Switch:SW_SPDT
Connections:
- net D14-Y2 (DL295) : now also U2.9 (A4); no longer U2.3 (A2)
- net STOP_CPU_WAIT: now also U2.8 (Y4); no longer U2.4 (Y2)
- net /AS (Host-CPU Pin9): now also U2.5 (A3); no longer U2.9 (A4)
- net at U1.4 (D): now also U2.6 (Y3); no longer U2.8 (Y4)
- new net: R102.1, SW1.2 (B)
- new net GNDD: SW1.3 (C)
- new net P3.2 (Host-CPU Pin12): R102.2
- new net P3.6 (BUSY, Video-CPU Pin40): SW1.1 (A)
Other:
- note added: "HINWEIS !!! Das BUSY-Signal der Video-CPU (P3.6, Pin40) sollte von P3.2 (Pin12) der Host-CPU getrennt und P3.2 dafür auf Masse gelegt werden, damit die Programme, welche das BUSY-Signal abfragen (z.B. die Grafik-Befehle des ES 4.0) schneller laufen."
- note removed: "HINWEIS !!! Das BUSY-Signal der Video-CPU (P3.6, Pin40) sollte von P3.2 (Pin12) der Host-CPU getrennt werden, damit die Programme, welche das BUSY-Signal abfragen (z.B. die Grafik-Befehle des ES 4.0) auch schneller laufen."
Changed lines of the file:
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@@
+    (stroke (width 0) (type default))
+  )
+  (wire (pts (xy 210.82 128.27) (xy 210.82 133.35))
     (stroke (width 0) (type default))
   )
@@
     (stroke (width 0) (type default))
   )
+  (wire (pts (xy 210.82 128.27) (xy 205.74 128.27))
+    (stroke (width 0) (type default))
+  )
   (wire (pts (xy 127 62.23) (xy 124.46 62.23))
     (stroke (width 0) (type default))
@@
     (stroke (width 0) (type default))
   )
+  (wire (pts (xy 180.34 125.73) (xy 184.15 125.73))
+    (stroke (width 0) (type default))
+  )
   (wire (pts (xy 96.52 58.42) (xy 111.76 58.42))
     (stroke (width 0) (type default))
@@
   )
   (wire (pts (xy 124.46 62.23) (xy 124.46 64.77))
+    (stroke (width 0) (type default))
+  )
+  (wire (pts (xy 205.74 123.19) (xy 215.9 123.19))
+    (stroke (width 0) (type default))
+  )
+  (wire (pts (xy 191.77 125.73) (xy 195.58 125.73))
     (stroke (width 0) (type default))
   )
@@
     (fill (type none))
   )
+  (rectangle (start 152.4 115.57) (end 255.27 138.43)
+    (stroke (width 0) (type dash) (color 194 0 0 1))
+    (fill (type none))
+  )
   (rectangle (start 60.96 35.56) (end 60.96 35.56)
     (stroke (width 0) (type default))
@@
     (effects (font (size 1.27 1.27) (color 194 0 0 1)) (justify left bottom))
   )
-  (text "HINWEIS !!!\n\nDas BUSY-Signal der Video-CPU (P3.6, Pin40) sollte von P3.2 (Pin12) \nder Host-CPU getrennt werden, damit die Programme, welche das BUSY-Signal \nabfragen (z.B. die Grafik-Befehle des ES 4.0) auch schneller laufen.\n\n "
-    (at 36.83 173.99 0)
+  (text "HINWEIS !!!\n\nDas BUSY-Signal der Video-CPU (P3.6, Pin40) sollte von P3.2 (Pin12) \nder Host-CPU getrennt und P3.2 dafür auf Masse gelegt werden, damit die \nProgramme, welche das BUSY-Signal abfragen (z.B. die Grafik-Befehle \ndes ES 4.0) schneller laufen. \n\n "
+    (at 152.4 156.21 0)
     (effects (font (size 1.27 1.27) (color 194 0 0 1)) (justify left bottom))
   )
@@
     (effects (font (size 1.27 1.27)) (justify left bottom))
   )
+  (global_label "P3.6 (BUSY, Video-CPU Pin40)" (shape input) (at 215.9 123.19 0) (fields_autoplaced)
+    (effects (font (size 1.27 1.27)) (justify left))
+    (property "Intersheetrefs" "${INTERSHEET_REFS}" (at 249.1649 123.19 0)
+      (effects (font (size 1.27 1.27)) (justify left) hide)
+    )
+  )
   (global_label "D14-Y2 (DL295) " (shape input) (at 63.5 116.84 180) (fields_autoplaced)
     (effects (font (size 1.27 1.27)) (justify right))
@@
     (effects (font (size 1.27 1.27)) (justify right))
     (property "Intersheetrefs" "${INTERSHEET_REFS}" (at 40.6975 105.41 0)
+      (effects (font (size 1.27 1.27)) (justify right) hide)
+    )
+  )
+  (global_label "P3.2 (Host-CPU Pin12)" (shape input) (at 180.34 125.73 180) (fields_autoplaced)
+    (effects (font (size 1.27 1.27)) (justify right))
+    (property "Intersheetrefs" "${INTERSHEET_REFS}" (at 154.3928 125.73 0)
       (effects (font (size 1.27 1.27)) (justify right) hide)
     )
@@
     )
   )
+  (symbol (lib_id "power:GNDD") (at 210.82 133.35 0) (unit 1)
+    (in_bom yes) (on_board yes) (dnp no) (fields_autoplaced)
+    (property "Reference" "#PWR02" (at 210.82 139.7 0)
+      (effects (font (size 1.27 1.27)) hide)
+    )
+    (property "Value" "GNDD" (at 210.82 138.43 0)
+      (effects (font (size 1.27 1.27)) hide)
+    )
+    (property "Footprint" "" (at 210.82 133.35 0)
+      (effects (font (size 1.27 1.27)) hide)
+    )
+    (property "Datasheet" "" (at 210.82 133.35 0)
+      (effects (font (size 1.27 1.27)) hide)
+    )
+    (pin "1")
+    (instances
+      (project "JU-TE-6K-Video-HW-Patch"
+        (path "/47571721-a842-4ec0-9206-b4e717bbb8bd"
+          (reference "#PWR02") (unit 1)
+        )
+      )
+    )
+  )
   (symbol (lib_id "RFT_Digitalschaltkreise:DL000D") (at 163.83 76.2 0) (unit 2)
     (in_bom yes) (on_board yes) (dnp no)
@@
     )
   )
-  (symbol (lib_id "RFT_Digitalschaltkreise:DL004D") (at 91.44 69.85 0) (unit 4)
+  (symbol (lib_id "RFT_Digitalschaltkreise:DL004D") (at 91.44 69.85 0) (unit 3)
     (in_bom yes) (on_board yes) (dnp no) (fields_autoplaced)
     (property "Reference" "U2" (at 91.6305 63.5 0)
@@
       (project "JU-TE-6K-Video-HW-Patch"
         (path "/47571721-a842-4ec0-9206-b4e717bbb8bd"
+          (reference "U2") (unit 3)
+        )
+      )
+    )
+  )
+  (symbol (lib_id "RFT_Digitalschaltkreise:DL004D") (at 91.44 58.42 0) (unit 2)
+    (in_bom yes) (on_board yes) (dnp no) (fields_autoplaced)
+    (property "Reference" "U2" (at 91.6305 52.07 0)
+      (effects (font (size 1.27 1.27)))
+    )
+    (property "Value" "DL004D" (at 91.6305 54.61 0)
+      (effects (font (size 1.27 1.27)))
+    )
+    (property "Footprint" "" (at 91.44 58.42 0)
+      (effects (font (size 1.27 1.27)) hide)
+    )
+    (property "Datasheet" "https://www-user.tu-chemnitz.de/~heha/basteln/Konsumg%C3%BCter/DDR-Halbleiter/dl003.gif" (at 91.44 64.77 0)
+      (effects (font (size 1.27 1.27)) hide)
+    )
+    (pin "2")
+    (pin "1")
+    (pin "3")
+    (pin "4")
+    (pin "5")
+    (pin "6")
+    (pin "8")
+    (pin "9")
+    (pin "10")
+    (pin "11")
+    (pin "12")
+    (pin "13")
+    (pin "14")
+    (pin "7")
+    (instances
+      (project "JU-TE-6K-Video-HW-Patch"
+        (path "/47571721-a842-4ec0-9206-b4e717bbb8bd"
+          (reference "U2") (unit 2)
+        )
+      )
+    )
+  )
+  (symbol (lib_id "Switch:SW_SPDT") (at 200.66 125.73 0) (unit 1)
+    (in_bom yes) (on_board yes) (dnp no)
+    (property "Reference" "SW1" (at 200.66 120.65 0)
+      (effects (font (size 1.27 1.27)))
+    )
+    (property "Value" "~" (at 200.66 121.92 0)
+      (effects (font (size 1.27 1.27)))
+    )
+    (property "Footprint" "" (at 200.66 125.73 0)
+      (effects (font (size 1.27 1.27)) hide)
+    )
+    (property "Datasheet" "~" (at 200.66 125.73 0)
+      (effects (font (size 1.27 1.27)) hide)
+    )
+    (pin "1")
+    (pin "2")
+    (pin "3")
+    (instances
+      (project "JU-TE-6K-Video-HW-Patch"
+        (path "/47571721-a842-4ec0-9206-b4e717bbb8bd"
+          (reference "SW1") (unit 1)
+        )
+      )
+    )
+  )
+  (symbol (lib_id "RFT_Digitalschaltkreise:DL004D") (at 82.55 116.84 0) (unit 4)
+    (in_bom yes) (on_board yes) (dnp no) (fields_autoplaced)
+    (property "Reference" "U2" (at 82.7405 110.49 0)
+      (effects (font (size 1.27 1.27)))
+    )
+    (property "Value" "DL004D" (at 82.7405 113.03 0)
+      (effects (font (size 1.27 1.27)))
+    )
+    (property "Footprint" "" (at 82.55 116.84 0)
+      (effects (font (size 1.27 1.27)) hide)
+    )
+    (property "Datasheet" "https://www-user.tu-chemnitz.de/~heha/basteln/Konsumg%C3%BCter/DDR-Halbleiter/dl003.gif" (at 82.55 123.19 0)
+      (effects (font (size 1.27 1.27)) hide)
+    )
+    (pin "2")
+    (pin "1")
+    (pin "3")
+    (pin "4")
+    (pin "5")
+    (pin "6")
+    (pin "8")
+    (pin "9")
+    (pin "10")
+    (pin "11")
+    (pin "12")
+    (pin "13")
+    (pin "14")
+    (pin "7")
+    (instances
+      (project "JU-TE-6K-Video-HW-Patch"
+        (path "/47571721-a842-4ec0-9206-b4e717bbb8bd"
           (reference "U2") (unit 4)
         )
@@
     )
   )
-  (symbol (lib_id "RFT_Digitalschaltkreise:DL004D") (at 91.44 58.42 0) (unit 2)
-    (in_bom yes) (on_board yes) (dnp no) (fields_autoplaced)
-    (property "Reference" "U2" (at 91.6305 52.07 0)
-      (effects (font (size 1.27 1.27)))
-    )
-    (property "Value" "DL004D" (at 91.6305 54.61 0)
-      (effects (font (size 1.27 1.27)))
-    )
-    (property "Footprint" "" (at 91.44 58.42 0)
-      (effects (font (size 1.27 1.27)) hide)
-    )
-    (property "Datasheet" "https://www-user.tu-chemnitz.de/~heha/basteln/Konsumg%C3%BCter/DDR-Halbleiter/dl003.gif" (at 91.44 64.77 0)
-      (effects (font (size 1.27 1.27)) hide)
-    )
-    (pin "2")
-    (pin "1")
-    (pin "3")
-    (pin "4")
-    (pin "5")
-    (pin "6")
-    (pin "8")
-    (pin "9")
-    (pin "10")
-    (pin "11")
-    (pin "12")
-    (pin "13")
-    (pin "14")
-    (pin "7")
-    (instances
-      (project "JU-TE-6K-Video-HW-Patch"
-        (path "/47571721-a842-4ec0-9206-b4e717bbb8bd"
-          (reference "U2") (unit 2)
-        )
-      )
-    )
-  )
-  (symbol (lib_id "RFT_Digitalschaltkreise:DL004D") (at 82.55 116.84 0) (unit 2)
-    (in_bom yes) (on_board yes) (dnp no) (fields_autoplaced)
-    (property "Reference" "U2" (at 82.7405 110.49 0)
-      (effects (font (size 1.27 1.27)))
-    )
-    (property "Value" "DL004D" (at 82.7405 113.03 0)
-      (effects (font (size 1.27 1.27)))
-    )
-    (property "Footprint" "" (at 82.55 116.84 0)
-      (effects (font (size 1.27 1.27)) hide)
-    )
-    (property "Datasheet" "https://www-user.tu-chemnitz.de/~heha/basteln/Konsumg%C3%BCter/DDR-Halbleiter/dl003.gif" (at 82.55 123.19 0)
-      (effects (font (size 1.27 1.27)) hide)
-    )
-    (pin "2")
-    (pin "1")
-    (pin "3")
-    (pin "4")
-    (pin "5")
-    (pin "6")
-    (pin "8")
-    (pin "9")
-    (pin "10")
-    (pin "11")
-    (pin "12")
-    (pin "13")
-    (pin "14")
-    (pin "7")
-    (instances
-      (project "JU-TE-6K-Video-HW-Patch"
-        (path "/47571721-a842-4ec0-9206-b4e717bbb8bd"
-          (reference "U2") (unit 2)
-        )
-      )
+  (symbol (lib_id "Device:R") (at 187.96 125.73 270) (unit 1)
+    (in_bom yes) (on_board yes) (dnp no) (fields_autoplaced)
+    (property "Reference" "R102" (at 187.96 120.65 90)
+      (effects (font (size 1.27 1.27)))
+    )
+    (property "Value" "10K" (at 187.96 123.19 90)
+      (effects (font (size 1.27 1.27)))
+    )
+    (property "Footprint" "" (at 187.96 123.952 90)
+      (effects (font (size 1.27 1.27)) hide)
+    )
+    (property "Datasheet" "~" (at 187.96 125.73 0)
+      (effects (font (size 1.27 1.27)) hide)
+    )
+    (pin "1")
+    (pin "2")
+    (instances
+      (project "JU-TE-6K-Video-HW-Patch"
+        (path "/47571721-a842-4ec0-9206-b4e717bbb8bd"
+          (reference "R102") (unit 1)
+        )
+      )
